File: rpglb_badge.sch (EAGLE design)
At the start: 151 parts

Commit message: Closer to finished schematic.
Parts:
- added BT1: (no value), SparkFun-Batteries:BATTERY-AA
- added C10, C11, C6, C7, C8, C9: 100nF, rcl:C-EUC0603
- added C12, C13: 4.7uF, rcl:C-EUC0603
- added C14, C15: 10uF, rcl:C-EUC0603
- added C16, C17: 1uF, rcl:C-EUC0603
- added C4, C5: 20pF, rcl:C-EUC0603
- added IC1: TS520550, v-reg:TS520550
- added J1: (no value), SparkFun-Connectors:USB_MICRO-B_SMT
- added L1: 4.5uH, rcl:L-USPIS2816
- added Q1: 8MHZ 10PF, crystal:CRYSTALCTS406
- added R2: 10K, rcl:R-EU_R0603
- added R3, R4: 1K, rcl:R-EU_R0603
- added S1, S2, S3, S4, S5, S6, S7, S8: MOMENTARY-SWITCH-SPST-SMD-5.2MM, SparkFun-Switches:MOMENTARY-SWITCH-SPST-SMD-5.2MM
- added S9: (no value), SparkFun-Switches:SWITCH-SPDT-SMD-RIGHT-ANGLE
- added U$3: TLV61225SOT6, konkers:TLV61225SOT6
- renumbered LED1 to LED1-1, LED10 to LED2-2, LED100 to LED4-12, LED101 to LED4-13, LED102 to LED4-14, LED103 to LED4-15, LED104 to LED4-16, LED105 to LED5-9, LED106 to LED5-10, LED107 to LED5-11, LED108 to LED5-12, LED109 to LED5-13, LED11 to LED2-3, LED110 to LED5-14, LED111 to LED5-15, LED112 to LED5-16, LED113 to LED6-9, LED114 to LED6-10, LED115 to LED6-11, LED116 to LED6-12, LED117 to LED6-13, LED118 to LED6-14, LED119 to LED6-15, LED12 to LED2-4, LED120 to LED6-16, LED121 to LED7-9, LED122 to LED7-10, LED123 to LED7-11, LED124 to LED7-12, LED125 to LED7-13, LED126 to LED7-14, LED127 to LED7-15, LED128 to LED7-16, LED129 to LED8-9, LED13 to LED2-5, LED130 to LED8-10, LED131 to LED8-11, LED132 to LED8-12, LED133 to LED8-13, LED134 to LED8-14, LED135 to LED8-15, LED136 to LED8-16, LED137 to LED9-9, LED138 to LED9-10, LED139 to LED9-11, LED14 to LED2-6, LED140 to LED9-12, LED141 to LED9-13, LED142 to LED9-14, LED143 to LED9-15, LED144 to LED9-16, LED15 to LED2-7, LED16 to LED2-8, LED17 to LED3-1, LED18 to LED3-2, LED19 to LED3-3, LED2 to LED1-2, LED20 to LED3-4, LED21 to LED3-5, LED22 to LED3-6, LED23 to LED3-7, LED24 to LED3-8, LED25 to LED4-1, LED26 to LED4-2, LED27 to LED4-3, LED28 to LED4-4, LED29 to LED4-5, LED3 to LED1-3, LED30 to LED4-6, LED31 to LED4-7, LED32 to LED4-8, LED33 to LED5-1, LED34 to LED5-2, LED35 to LED5-3, LED36 to LED5-4, LED37 to LED5-5, LED38 to LED5-6, LED39 to LED5-7, LED4 to LED1-4, LED40 to LED5-8, LED41 to LED6-1, LED42 to LED6-2, LED43 to LED6-3, LED44 to LED6-4, LED45 to LED6-5, LED46 to LED6-6, LED47 to LED6-7, LED48 to LED6-8, LED49 to LED7-1, LED5 to LED1-5, LED50 to LED7-2, LED51 to LED7-3, LED52 to LED7-4, LED53 to LED7-5, LED54 to LED7-6, LED55 to LED7-7, LED56 to LED7-8, LED57 to LED8-1, LED58 to LED8-2, LED59 to LED8-3, LED6 to LED1-6, LED60 to LED8-4, LED61 to LED8-5, LED62 to LED8-6, LED63 to LED8-7, LED64 to LED8-8, LED65 to LED9-1, LED66 to LED9-2, LED67 to LED9-3, LED68 to LED9-4, LED69 to LED9-5, LED7 to LED1-7, LED70 to LED9-6, LED71 to LED9-7, LED72 to LED9-8, LED73 to LED1-9, LED74 to LED1-10, LED75 to LED1-11, LED76 to LED1-12, LED77 to LED1-13, LED78 to LED1-14, LED79 to LED1-15, LED8 to LED1-8, LED80 to LED1-16, LED81 to LED2-9, LED82 to LED2-10, LED83 to LED2-11, LED84 to LED2-12, LED85 to LED2-13, LED86 to LED2-14, LED87 to LED2-15, LED88 to LED2-16, LED89 to LED3-9, LED9 to LED2-1, LED90 to LED3-10, LED91 to LED3-11, LED92 to LED3-12, LED93 to LED3-13, LED94 to LED3-14, LED95 to LED3-15, LED96 to LED3-16, LED97 to LED4-9, LED98 to LED4-10, LED99 to LED4-11
Connections:
- new net B_A: S7.1, U$2.PA4
- new net B_B: S8.1, U$2.PA5
- new net B_DOWN: S4.1, U$2.PA1
- new net B_LEFT: S5.1, U$2.PA2
- new net B_RIGHT: S6.1, U$2.PA3
- new net B_UP: S3.1, U$2.PA0
- new net N$3: C5.1, Q1.2, U$2.PF1_OSC_OUT
- new net N$4: C4.1, Q1.1, U$2.PF0_OSC_IN
- new net N$5: C6.2, R2.2, S2.1, U$2.BOOT0
- new net N$6: L1.2, U$3.L
- new net SCL: R3.1, U$2.PB10
- new net UART_RX: U$2.PA10
- new net UART_TX: U$2.PA9
- new net USB_DM: J1.D-, U$2.PA11
- new net USB_DP: J1.D+, U$2.PA12
- new net V33_BATT: C14.1, S9.S, U$3.FB, U$3.VOUT
- new net V33_USB: C17.1, IC1.VOUT, S9.O
- new net V_BATT: BT1.+, C15.1, L1.1, U$3.EN, U$3.VIN
- new net V_USB: C16.1, IC1.CE, IC1.VIN, J1.VBUS
- net +3V3: now also C10.1, C11.1, C12.1, C13.1, C6.1, C8.1, C9.1, R3.2, R4.2, S2.2, S9.P
- net GND: now also BT1.-, C10.2, C11.2, C12.2, C13.2, C14.2, C15.2, C16.2, C17.2, C4.2, C5.2, C7.2, C8.2, C9.2, J1.GND, R2.1, S1.1, S3.2, S4.2, S5.2, S6.2, S7.2, S8.2, U$3.GND
- net NRST: now also C7.1, S1.2
- net SDA: now also R4.1, U$2.PB11
Other:
- note added: "VDD decaps"
- note added: "VDDIO2 decaps"
